Commit message: 260514 gripper and box in gazebo

File: cra_description/urdf/cr7_robot.xacro (robot description, xacro)
@@ -1,4 +1,5 @@
 <?xml version="1.0"?>
 <robot name="cr7_robot"  xmlns:xacro="http://ros.org/wiki/xacro">
+  <xacro:include filename="$(find cra_description)/urdf/gripper.xacro"/>
     <link name="dummy_link" />
   <link name="base_link">
@@ -426,5 +427,7 @@
         <selfCollide>true</selfCollide>
     </gazebo>
-    <!-- 在运行demo.launch.py时，需要注释这个ros2_control节点，因为它使用了xxx.ros2_control.xacro来生成了ros2_control节点-->
+    <xacro:simple_gripper parent="Link6" prefix="">
+      <origin xyz="0 0 0" rpy="0 0 0"/>
+    </xacro:simple_gripper>
     <ros2_control name="GazeboSystem" type="system">
         <hardware>
@@ -490,4 +493,22 @@
             </state_interface>
             <state_interface name="velocity"/>
+        </joint>
+        <joint name="left_finger_joint">
+            <command_interface name="position">
+                <param name="min">0.0</param>
+                <param name="max">0.080</param>
+            </command_interface>
+            <state_interface name="position"/>
+            <state_interface name="velocity"/>
+            <state_interface name="effort"/>
+        </joint>
+        <joint name="right_finger_joint">
+            <command_interface name="position">
+                <param name="min">0.0</param>
+                <param name="max">0.080</param>
+            </command_interface>
+            <state_interface name="position"/>
+            <state_interface name="velocity"/>
+            <state_interface name="effort"/>
         </joint>
     </ros2_control>

Commit message: 260602 first pick and place with gripper pose holding

File: cra_description/urdf/cr7_robot.xacro (robot description, xacro)
@@ -1,5 +1,5 @@
 <?xml version="1.0"?>
 <robot name="cr7_robot"  xmlns:xacro="http://ros.org/wiki/xacro">
-  <xacro:include filename="$(find cra_description)/urdf/gripper.xacro"/>
+  <xacro:include filename="$(find onrobot_2fg7_description)/urdf/onrobot_2fg7.xacro"/>
     <link name="dummy_link" />
   <link name="base_link">
@@ -427,7 +427,39 @@
         <selfCollide>true</selfCollide>
     </gazebo>
-    <xacro:simple_gripper parent="Link6" prefix="">
+    <!-- OnRobot 2FG7 gripper attached to Link6 -->
+    <xacro:onrobot_2fg7 prefix="gripper_" parent="Link6">
       <origin xyz="0 0 0" rpy="0 0 0"/>
-    </xacro:simple_gripper>
+    </xacro:onrobot_2fg7>
+    <xacro:onrobot_2fg7_fingertip prefix="gripper_right_" parent="gripper_right_attachment">
+      <origin xyz="0 0 0" rpy="0 0 3.14159265359"/>
+    </xacro:onrobot_2fg7_fingertip>
+    <xacro:onrobot_2fg7_fingertip prefix="gripper_left_" parent="gripper_left_attachment">
+      <origin xyz="0 0 0" rpy="0 0 0"/>
+    </xacro:onrobot_2fg7_fingertip>
+    <!-- Gazebo settings for gripper links (blue base, yellow fingers, no gravity, grip contact tuning) -->
+    <gazebo reference="gripper_base_link">
+        <material>Gazebo/Blue</material>
+        <gravity>false</gravity>
+    </gazebo>
+    <gazebo reference="gripper_right_onrobot_2fg7_finger_link">
+        <material>Gazebo/Yellow</material>
+        <gravity>false</gravity>
+        <mu1>100.0</mu1>
+        <mu2>100.0</mu2>
+        <kp>200000.0</kp>
+        <kd>10.0</kd>
+        <minDepth>0.002</minDepth>
+        <maxVel>0.05</maxVel>
+    </gazebo>
+    <gazebo reference="gripper_left_onrobot_2fg7_finger_link">
+        <material>Gazebo/Yellow</material>
+        <gravity>false</gravity>
+        <mu1>100.0</mu1>
+        <mu2>100.0</mu2>
+        <kp>200000.0</kp>
+        <kd>10.0</kd>
+        <minDepth>0.002</minDepth>
+        <maxVel>0.05</maxVel>
+    </gazebo>
     <ros2_control name="GazeboSystem" type="system">
         <hardware>
@@ -494,19 +526,23 @@
             <state_interface name="velocity"/>
         </joint>
-        <joint name="left_finger_joint">
-            <command_interface name="position">
-                <param name="min">0.0</param>
-                <param name="max">0.080</param>
-            </command_interface>
-            <state_interface name="position"/>
+        <joint name="gripper_gripper_joint">
+            <command_interface name="position">
+                <param name="min">0.0115</param>
+                <param name="max">0.10</param>
+            </command_interface>
+            <state_interface name="position">
+                <param name="initial_value">0.0115</param>
+            </state_interface>
             <state_interface name="velocity"/>
             <state_interface name="effort"/>
         </joint>
-        <joint name="right_finger_joint">
-            <command_interface name="position">
-                <param name="min">0.0</param>
-                <param name="max">0.080</param>
-            </command_interface>
-            <state_interface name="position"/>
+        <joint name="gripper_right_finger_joint">
+            <command_interface name="position">
+                <param name="min">0.0115</param>
+                <param name="max">0.10</param>
+            </command_interface>
+            <state_interface name="position">
+                <param name="initial_value">0.0115</param>
+            </state_interface>
             <state_interface name="velocity"/>
             <state_interface name="effort"/>
