Commit message: 260709 all sequence(no vision) & mcs comm

File: src/DOBOT_6Axis_ROS2_V4/cra_description/urdf/arm_on_mpo700.urdf.xacro (robot description, xacro)
@@ -6,8 +6,9 @@
      The CR7 root link is kept named "base_link" so cbirrt_pick_place.py
      (frame_id="base_link") and the MoveIt config keep working unchanged. -->
-<robot name="cr7_on_mpo700" xmlns:xacro="http://www.ros.org/wiki/xacro">
+<robot name="arm_on_mpo700" xmlns:xacro="http://www.ros.org/wiki/xacro">
   <!-- Args required by the imported MPO-700 description -->
   <xacro:arg name="use_gazebo" default="true"/>
   <xacro:arg name="use_docking_adapter" default="false"/>
+  <xacro:arg name="arm_type" default="cr10"/>
   <!-- OmniDriveModule joint type (fixed for simulation) -->
   <xacro:property name="ODM_joint_type" value="fixed"/>
@@ -121,196 +122,10 @@
     <child link="base_link"/>
   </joint>
-  <!-- ===================== CR7 arm ===================== -->
-  <link name="base_link">
-    <inertial>
-      <origin xyz="-7.75881826404344E-06 0.00191109737802069 0.0289949710713939" rpy="0 0 0" />
-      <mass value="0.908795453638862" />
-      <inertia ixx="0.00145446136430631" ixy="4.10411509661615E-08" ixz="-1.83603068187756E-07"
-               iyy="0.00134497445765809" iyz="-6.24662501711042E-06" izz="0.00215495523232905" />
-    </inertial>
-    <visual>
-      <origin xyz="0 0 0" rpy="0 0 0" />
-      <geometry>
-        <mesh filename="file://$(find cra_description)/meshes/cr7/base_link0.STL" />
-      </geometry>
-      <material name="cr7_silver">
-        <color rgba="0.792156862745098 0.819607843137255 0.933333333333333 1" />
-      </material>
-    </visual>
-    <collision>
-      <origin xyz="0 0 0" rpy="0 0 0" />
-      <geometry>
-        <mesh filename="file://$(find cra_description)/meshes/cr7/base_link0.STL" />
-      </geometry>
-    </collision>
-  </link>
-  <link name="Link1">
-    <inertial>
-      <origin xyz="2.42083892138974E-07 -0.00325669708857515 -0.00767435596457115" rpy="0 0 0" />
-      <mass value="1.6123155679073" />
-      <inertia ixx="0.00291211377650885" ixy="-7.47419584239082E-09" ixz="1.94780650217368E-08"
-               iyy="0.00281918869862419" iyz="0.000440963272842605" izz="0.00328358201221721" />
-    </inertial>
-    <visual>
-      <origin xyz="0 0 0" rpy="0 0 0" />
-      <geometry>
-        <mesh filename="file://$(find cra_description)/meshes/cr7/J1.STL" />
-      </geometry>
-      <material name="cr7_silver"/>
-    </visual>
-    <collision>
-      <origin xyz="0 0 0" rpy="0 0 0" />
-      <geometry>
-        <mesh filename="file://$(find cra_description)/meshes/cr7/J1.STL" />
-      </geometry>
-    </collision>
-  </link>
-  <joint name="joint1" type="revolute">
-    <origin xyz="0 0 0.147" rpy="0 0 0" />
-    <parent link="base_link" />
-    <child link="Link1" />
-    <axis xyz="0 0 -1" />
-    <limit lower="-6.27" upper="6.27" effort="300" velocity="100" />
-  </joint>
-  <link name="Link2">
-    <inertial>
-      <origin xyz="-0.188500103625708 -7.46110088887752E-07 0.142319304936727" rpy="0 0 0" />
-      <mass value="5.28764336862191" />
-      <inertia ixx="0.00860086052884714" ixy="3.30521626209469E-09" ixz="-4.99788929762243E-09"
-               iyy="0.0181761454963347" iyz="-1.56481985512198E-08" izz="0.0189188799857172" />
-    </inertial>
-    <visual>
-      <origin xyz="0 0 0" rpy="0 0 0" />
-      <geometry>
-        <mesh filename="file://$(find cra_description)/meshes/cr7/J2.STL" />
-      </geometry>
-      <material name="cr7_silver"/>
-    </visual>
-    <collision>
-      <origin xyz="0 0 0" rpy="0 0 0" />
-      <geometry>
-        <mesh filename="file://$(find cra_description)/meshes/cr7/J2.STL" />
-      </geometry>
-    </collision>
-  </link>
-  <joint name="joint2" type="revolute">
-    <origin xyz="0 0 0" rpy="-1.57080420997483 1.57079631189374 -3.14158502419526" />
-    <parent link="Link1" />
-    <child link="Link2" />
-    <axis xyz="0 0 1" />
-    <limit lower="-6.27" upper="6.27" effort="300" velocity="100" />
-  </joint>
-  <link name="Link3">
-    <inertial>
-      <origin xyz="-0.129084033261017 0.000409825982416691 -0.0024891265183234" rpy="0 0 0" />
-      <mass value="2.64536322797469" />
-      <inertia ixx="0.00313429310657436" ixy="8.58567214179718E-06" ixz="0.0001236219933347"
-               iyy="0.00583755221707048" iyz="-3.84538201491329E-07" izz="0.00609610718076456" />
-    </inertial>
-    <visual>
-      <origin xyz="0 0 0" rpy="0 0 0" />
-      <geometry>
-        <mesh filename="file://$(find cra_description)/meshes/cr7/J3.STL" />
-      </geometry>
-      <material name="cr7_silver"/>
-    </visual>
-    <collision>
-      <origin xyz="0 0 0" rpy="0 0 0" />
-      <geometry>
-        <mesh filename="file://$(find cra_description)/meshes/cr7/J3.STL" />
-      </geometry>
-    </collision>
-  </link>
-  <joint name="joint3" type="revolute">
-    <origin xyz="-0.377 0 0.025" rpy="0 0 0" />
-    <parent link="Link2" />
-    <child link="Link3" />
-    <axis xyz="0 0 1" />
-    <limit lower="-2.79" upper="2.79" effort="300" velocity="100" />
-  </joint>
-  <link name="Link4">
-    <inertial>
-      <origin xyz="-0.00098049161725656 -0.00207570116557487 -0.00155508673006152" rpy="0 0 0" />
-      <mass value="0.670573134819647" />
-      <inertia ixx="0.000669371731621344" ixy="-5.32805461934157E-08" ixz="3.52586632357936E-07"
-               iyy="0.000654228488306913" iyz="0.000110801103983602" izz="0.000653654751027863" />
-    </inertial>
-    <visual>
-      <origin xyz="0 0 0" rpy="0 0 0" />
-      <geometry>
-        <mesh filename="file://$(find cra_description)/meshes/cr7/J4.STL" />
-      </geometry>
-      <material name="cr7_silver"/>
-    </visual>
-    <collision>
-      <origin xyz="0 0 0" rpy="0 0 0" />
-      <geometry>
-        <mesh filename="file://$(find cra_description)/meshes/cr7/J4.STL" />
-      </geometry>
-    </collision>
-  </link>
-  <joint name="joint4" type="revolute">
-    <origin xyz="-0.306999999999969 0 0.116" rpy="0 0 -1.57079677671549" />
-    <parent link="Link3" />
-    <child link="Link4" />
-    <axis xyz="0 0 0.999999999969965" />
-    <limit lower="-6.27" upper="6.27" effort="300" velocity="100" />
-  </joint>
-  <link name="Link5">
-    <inertial>
-      <origin xyz="-0.00139233872001005 -0.00449255371185306 -0.00130478579616922" rpy="0 0 0" />
-      <mass value="0.725828190120638" />
-      <inertia ixx="0.00073002940905788" ixy="1.46530702319641E-07" ixz="-1.21461719923983E-07"
-               iyy="0.000710023403641111" iyz="-0.000119103387993809" izz="0.000712169450212708" />
-    </inertial>
-    <visual>
-      <origin xyz="0 0 0" rpy="0 0 0" />
-      <geometry>
-        <mesh filename="file://$(find cra_description)/meshes/cr7/J5.STL" />
-      </geometry>
-      <material name="cr7_silver"/>
-    </visual>
-    <collision>
-      <origin xyz="0 0 0" rpy="0 0 0" />
-      <geometry>
-        <mesh filename="file://$(find cra_description)/meshes/cr7/J5.STL" />
-      </geometry>
-    </collision>
-  </link>
-  <joint name="joint5" type="revolute">
-    <origin xyz="0 -0.116 0" rpy="1.5707963267949 0 0" />
-    <parent link="Link4" />
-    <child link="Link5" />
-    <axis xyz="0 0 -1" />
-    <limit lower="-6.27" upper="6.27" effort="300" velocity="100" />
-  </joint>
-  <link name="Link6">
-    <inertial>
-      <origin xyz="-0.00134099075400824 9.61028193323665E-05 -0.0192856508049091" rpy="0 0 0" />
-      <mass value="0.157885328078873" />
-      <inertia ixx="7.80450650011017E-05" ixy="3.56327806101489E-09" ixz="-3.98217377472077E-11"
-               iyy="7.91678595101433E-05" iyz="-1.3821786505554E-07" izz="0.000129505866960959" />
-    </inertial>
-    <visual>
-      <origin xyz="0 0 0" rpy="0 0 0" />
-      <geometry>
-        <mesh filename="file://$(find cra_description)/meshes/cr7/J6.STL" />
-      </geometry>
-      <material name="cr7_silver"/>
-    </visual>
-    <collision>
-      <origin xyz="0 0 0" rpy="0 0 0" />
-      <geometry>
-        <mesh filename="file://$(find cra_description)/meshes/cr7/J6.STL" />
-      </geometry>
-    </collision>
-  </link>
-  <joint name="joint6" type="revolute">
-    <origin xyz="0 0.104999656773681 0" rpy="-1.5707963267949 0 0" />
-    <parent link="Link5" />
-    <child link="Link6" />
-    <axis xyz="0 0 -1" />
-    <limit lower="-6.27" upper="6.27" effort="300" velocity="100" />
-  </joint>
+  <!-- ===================== Arm (swappable) ===================== -->
+  <!-- arm_type picks {arm_type}_arm.xacro (base_link + Link1..6 + joint1..6).
+       Default cr10; override via launch arg / run_mpo700_<arm>.sh. All Dobot CR
+       arms share joint names (joint1..6) and root link base_link, so the cube
+       mount, ros2_control, gripper and camera below stay arm-agnostic. -->
+  <xacro:include filename="$(find cra_description)/urdf/$(arg arm_type)_arm.xacro"/>
   <!-- Base + cube: no gravity. The AGV is velocity-controlled by the planar-move
        plugin (it does not rely on weight/wheel friction) and the arm is
@@ -386,9 +201,7 @@
       <material name="d405_alu"><color rgba="0.7 0.72 0.75 1"/></material>
     </visual>
-    <!-- Camera collision DISABLED on purpose: the D405 body at the wrist kept
-         blocking tight slot approaches (planner) and snagging the device (Gazebo).
-         The camera is a sensor, not a structural part; the wrist/gripper collision
-         geometry still guards this region. Restore the block below if a real-robot
-         deployment needs the camera body protected.
+    <!-- Camera collision DISABLED on purpose, same as cr7_on_mpo700.urdf.xacro:
+         the D405 body kept blocking tight slot approaches; the wrist/gripper
+         collision geometry still guards this region. Restore for real-robot use.
     <collision>
       <origin xyz="0 0 0" rpy="1.5707963 0 1.5707963"/>
@@ -437,13 +250,20 @@
   </gazebo>
   <!-- ===================== CR7 ros2_control ===================== -->
+  <!-- Per-arm tool-down standby (initial joint values). Same joint angles give a
+       DIFFERENT pose on each arm (link lengths / joint frames differ), so the start
+       pose is keyed on arm_type. cr10: collision-checked tool-down (tool z = world
+       -Z, TCP in front). Unknown arms fall back to all-zeros (may not be tool-down;
+       add an entry to init_q when porting cr12/16/20). -->
+  <xacro:property name="arm_type" value="$(arg arm_type)"/>
+  <xacro:if value="${arm_type == 'cr10'}">
+    <xacro:property name="init_q" value="${[-0.7739, -0.0178, -2.4042, 0.9124, 1.5762, 0.8885]}"/>
+  </xacro:if>
+  <xacro:unless value="${arm_type == 'cr10'}">
+    <xacro:property name="init_q" value="${[0.0, 0.0, 0.0, 0.0, 0.0, 0.0]}"/>
+  </xacro:unless>
   <ros2_control name="GazeboSystem" type="system">
     <hardware>
       <plugin>gazebo_ros2_control/GazeboSystem</plugin>
     </hardware>
-    <!-- Spawn AT the hub (tool-down standby, TCP=(0.33,0,0.32)): the same pose
-         wirebonder_pick_place.py drives to with go_to_hub() at startup. Spawning
-         here means the arm never has to swing from a folded/upright pose into the
-         hub on bring-up. Joints (rad) from _calc_hub_q.py (project IK, collision-
-         gated): J1..J6 deg = -26.0,+19.7,-107.9,0,-87.4,-24.7. -->
     <joint name="joint1">
       <command_interface name="position">
@@ -452,5 +272,5 @@
       </command_interface>
       <state_interface name="position">
-        <param name="initial_value">-0.45320</param>
+        <param name="initial_value">${init_q[0]}</param>
       </state_interface>
       <state_interface name="velocity"/>
@@ -462,5 +282,5 @@
       </command_interface>
       <state_interface name="position">
-        <param name="initial_value">0.34299</param>
+        <param name="initial_value">${init_q[1]}</param>
       </state_interface>
       <state_interface name="velocity"/>
@@ -472,5 +292,5 @@
       </command_interface>
       <state_interface name="position">
-        <param name="initial_value">-1.88375</param>
+        <param name="initial_value">${init_q[2]}</param>
       </state_interface>
       <state_interface name="velocity"/>
@@ -482,5 +302,5 @@
       </command_interface>
       <state_interface name="position">
-        <param name="initial_value">0.0</param>
+        <param name="initial_value">${init_q[3]}</param>
       </state_interface>
       <state_interface name="velocity"/>
@@ -492,5 +312,5 @@
       </command_interface>
       <state_interface name="position">
-        <param name="initial_value">-1.52609</param>
+        <param name="initial_value">${init_q[4]}</param>
       </state_interface>
       <state_interface name="velocity"/>
@@ -502,5 +322,5 @@
       </command_interface>
       <state_interface name="position">
-        <param name="initial_value">-0.43032</param>
+        <param name="initial_value">${init_q[5]}</param>
       </state_interface>
       <state_interface name="velocity"/>

Commit message: 260716 All sequences(shelf, teleop_agv, wirebonding) success!

File: src/DOBOT_6Axis_ROS2_V4/cra_description/urdf/arm_on_mpo700.urdf.xacro (robot description, xacro)
@@ -197,5 +197,5 @@
       <origin xyz="0 0 0" rpy="1.5707963 0 1.5707963"/>
       <geometry>
-        <mesh filename="file:///home/user/dobot_ws/src/realsense-ros/realsense2_description/meshes/d405.stl" scale="0.001 0.001 0.001"/>
+        <mesh filename="file://$(find cra_description)/meshes/d405.stl" scale="0.001 0.001 0.001"/>
       </geometry>
       <material name="d405_alu"><color rgba="0.7 0.72 0.75 1"/></material>
@@ -207,5 +207,5 @@
       <origin xyz="0 0 0" rpy="1.5707963 0 1.5707963"/>
       <geometry>
-        <mesh filename="file:///home/user/dobot_ws/src/realsense-ros/realsense2_description/meshes/d405.stl" scale="0.001 0.001 0.001"/>
+        <mesh filename="file://$(find cra_description)/meshes/d405.stl" scale="0.001 0.001 0.001"/>
       </geometry>
     </collision>

File: src/DOBOT_6Axis_ROS2_V4/cra_description/urdf/cr7_mpo700_body.urdf.xacro (robot description, xacro)
@@ -4,7 +4,10 @@
     <link name="mpo_base_link">
         <inertial>
-            <mass value="140"/>
+            <!-- x10 (2026-07-16), with the cube_link ballast bump: shrink the
+                 contact-impulse ratchet. planar_move drives by velocity, so
+                 teleop is unaffected. -->
+            <mass value="1400"/>
             <origin xyz="0 0 0"/>
-            <inertia ixx="7.8" ixy="0.0" ixz="0" iyy="7.8" iyz="0.0" izz="7.8"/>
+            <inertia ixx="78" ixy="0.0" ixz="0" iyy="78" iyz="0.0" izz="78"/>
         </inertial>
         <visual>

File: src/DOBOT_6Axis_ROS2_V4/cra_description/urdf/cr7_on_mpo700.urdf.xacro (robot description, xacro)
@@ -38,8 +38,14 @@
          never enters the purely kinematic IK or collision checks); it only
          changes Gazebo physics. -->
-    <inertial>
-      <mass value="500.0"/>
+    <!-- x10 ballast bump (2026-07-16): 500 kg / I=2000 still ratcheted a few
+         mm-deg per cycle (no restoring force, so every impulse leaves a
+         residue). With x10 the same impulses leave ~1/10 the residue; combined
+         with the guarded pocket place (no more 5 mm press) the per-cycle drift
+         should be sub-mm, replacing the level_base teleport calls. Driving is
+         unaffected: planar_move commands VELOCITY, not force. -->
+    <inertial>
+      <mass value="5000.0"/>
       <origin xyz="0 0 -0.35" rpy="0 0 0"/>
-      <inertia ixx="2000.0" ixy="0" ixz="0" iyy="2000.0" iyz="0" izz="2000.0"/>
+      <inertia ixx="20000.0" ixy="0" ixz="0" iyy="20000.0" iyz="0" izz="20000.0"/>
     </inertial>
     <!-- Front half (+X): robot mounting area, 0.3705 x 0.509 x 0.66 m
@@ -317,8 +323,11 @@
        still RATCHET from contact impulses regardless of gravity, because
        gazebo_ros_planar_move zeroes angular-x/y and linear-z velocity every tick
-       (no restoring path; gravity-on was tried and changed nothing). The shelf
-       sequence therefore re-LEVELS the base by teleport at each park
-       (shelf_pick_place._level_base), a sim-only workaround; the real AGV's
-       mass/suspension makes this failure class physically impossible. -->
+       (no restoring path; gravity-on was tried and changed nothing). Treatment
+       history: per-cycle level_base teleports (2026-07-15) were RETIRED on
+       2026-07-16 in favour of the x10 ballast bump (cube_link inertial below;
+       mpo_base_link in cr7_mpo700_body.urdf.xacro), which shrinks the
+       per-impulse residue ~x10; node.level_base remains available as a manual
+       repair. The real AGV's mass/suspension makes this failure class
+       physically impossible. -->
   <gazebo reference="mpo_base_link">
     <gravity>false</gravity>
@@ -389,5 +398,5 @@
       <origin xyz="0 0 0" rpy="1.5707963 0 1.5707963"/>
       <geometry>
-        <mesh filename="file:///home/user/dobot_ws/src/realsense-ros/realsense2_description/meshes/d405.stl" scale="0.001 0.001 0.001"/>
+        <mesh filename="file://$(find cra_description)/meshes/d405.stl" scale="0.001 0.001 0.001"/>
       </geometry>
       <material name="d405_alu"><color rgba="0.7 0.72 0.75 1"/></material>
@@ -401,5 +410,5 @@
       <origin xyz="0 0 0" rpy="1.5707963 0 1.5707963"/>
       <geometry>
-        <mesh filename="file:///home/user/dobot_ws/src/realsense-ros/realsense2_description/meshes/d405.stl" scale="0.001 0.001 0.001"/>
+        <mesh filename="file://$(find cra_description)/meshes/d405.stl" scale="0.001 0.001 0.001"/>
       </geometry>
     </collision>
@@ -407,5 +416,17 @@
   </link>
   <joint name="d405_joint" type="fixed">
-    <origin xyz="0.071 0 0.147" rpy="0 0 0"/>
+    <!-- Fixed-jaw bend mount (adopted 2026-07-15): camera back FLUSH on the
+         jaw bend front face, top level with the jaw arm top. NOTE the
+         d405_link origin is the LENS FACE and the body extends 23 mm BEHIND it
+         (measured from d405.stl): origin x = jaw front face (0.2009,
+         jaw_fixed.stl) + 23 mm = 0.2239; origin z = jaw arm top (0.115) -
+         42mm/2 = 0.094. Body spans x[0.2009, 0.2239] z[0.073, 0.115]: flush
+         with the jaw, clear of pads and the carried box (box x <= 0.182).
+         Validated: tag capture 50 px at CAPTURE_A_JOINTS, anchor read within
+         0.5 mm (no OLD_DEVICE_POSE recapture needed in sim), pocket
+         LOOK_JOINTS re-jogged. Old top-plate mount: xyz="0.071 0 0.147".
+         REAL ROBOT: hand-eye cal + OLD_DEVICE_POSE recapture after mounting
+         (docs/real_robot_transition.md). -->
+    <origin xyz="0.2239 0 0.094" rpy="0 0 0"/>
     <parent link="gripper_base_link"/>
     <child link="d405_link"/>

File: src/DOBOT_6Axis_ROS2_V4/cra_description/urdf/gripper.xacro (robot description, xacro)
@@ -11,5 +11,5 @@
        Gazebo-sim robots; false for the MoveIt-only description, which has none). -->
   <xacro:macro name="cr7_gripper" params="gazebo_props:=true">
-    <xacro:property name="mesh" value="file:///home/user/dobot_ws/src/blender/gripper_long"/>
+    <xacro:property name="mesh" value="file://$(env HOME)/dobot_ws/src/blender/gripper_long"/>
     <!-- Fixed part: flange + body + integral L-jaw + fixed pad -->
     <link name="gripper_base_link">
