Commit message: 260619 shelf-base full cycle with long gripper

File: src/DOBOT_6Axis_ROS2_V4/cr7_moveit/config/cr7_robot.urdf.xacro (robot description, xacro)
@@ -1,61 +1,15 @@
 <?xml version="1.0"?>
-<robot xmlns:xacro="http://www.ros.org/wiki/xacro" name="cr7_robot">
+<!-- Robot name MUST match the Gazebo robot_state_publisher model (cr7_on_mpo700)
+     so move_group's published planning scene is not rejected by RViz with
+     "Setting the scene for model 'cr7_robot' but model 'cr7_on_mpo700' is loaded".
+     This URDF is still arm+gripper only (no AGV/cube); only the name is shared. -->
+<robot xmlns:xacro="http://www.ros.org/wiki/xacro" name="cr7_on_mpo700">
     <xacro:arg name="initial_positions_file" default="initial_positions.yaml" />
     <!-- Import cr7_robot urdf file -->
     <xacro:include filename="$(find dobot_rviz)/urdf/cr7_robot.urdf" />
-    <!-- Blender fixed-jaw gripper (kinematics/collision only, no gazebo tags).
-         The dobot_rviz URDF above is the bare arm, but the Gazebo
-         joint_state_broadcaster publishes gripper_finger_joint on /joint_states;
-         without these links move_group logs "Joint 'gripper_finger_joint' not
-         found in model 'cr7_robot'" for every incoming message. Geometry copied
-         from cra_description/urdf/cr7_on_mpo700.urdf.xacro; keep in sync. -->
-    <link name="gripper_base_link">
-      <visual>
-        <origin xyz="0 0 0" rpy="0 0 0"/>
-        <geometry>
-          <mesh filename="file:///home/user/dobot_ws/src/blender/gripper/meshes/base.dae"/>
-        </geometry>
-      </visual>
-      <collision>  <!-- fixed-jaw top beam: X[0.009,0.107] Y[+-0.046] Z[0.105,0.115] -->
-        <origin xyz="0.0581 0 0.110" rpy="0 0 0"/>
-        <geometry><box size="0.098 0.0912 0.010"/></geometry>
-      </collision>
-      <collision>  <!-- fixed-jaw column + pad: X[0.0894,0.1071] Y[+-0.046] Z[0.055,0.105] -->
-        <origin xyz="0.0983 0 0.080" rpy="0 0 0"/>
-        <geometry><box size="0.0177 0.0912 0.050"/></geometry>
-      </collision>
-      <collision>  <!-- top plate (Cube_071): X[+-0.061] Y[+-0.046] Z[0.115,0.127] -->
-        <origin xyz="0 0 0.121" rpy="0 0 0"/>
-        <geometry><box size="0.121 0.091 0.012"/></geometry>
-      </collision>
-      <collision>  <!-- mount boss (Cylinder_004): r0.041 at Z[0.127,0.140] -->
-        <origin xyz="0 0 0.134" rpy="0 0 0"/>
-        <geometry><cylinder radius="0.041" length="0.013"/></geometry>
-      </collision>
-    </link>
-    <joint name="gripper_attach_joint" type="fixed">
-      <origin xyz="0 0 0.1401" rpy="3.14159265359 0 0"/>
-      <parent link="Link6"/>
-      <child link="gripper_base_link"/>
-    </joint>
-    <link name="gripper_finger_link">
-      <visual>
-        <origin xyz="0 0 0" rpy="0 0 0"/>
-        <geometry>
-          <mesh filename="file:///home/user/dobot_ws/src/blender/gripper/meshes/finger.dae"/>
-        </geometry>
-      </visual>
-      <collision>  <!-- moving jaw + pad: X[-0.011,0.016] Y[+-0.035] Z[0.056,0.127] -->
-        <origin xyz="0.0025 0 0.0915" rpy="0 0 0"/>
-        <geometry><box size="0.027 0.070 0.071"/></geometry>
-      </collision>
-    </link>
-    <joint name="gripper_finger_joint" type="prismatic">
-      <origin xyz="0 0 0" rpy="0 0 0"/>
-      <parent link="gripper_base_link"/>
-      <child link="gripper_finger_link"/>
-      <axis xyz="-1 0 0"/>
-      <limit lower="-0.07" upper="0.10" effort="60" velocity="0.1"/>
-    </joint>
+    <!-- Gripper: single source of truth in cra_description/urdf/gripper.xacro.
+         MoveIt-only description -> no Gazebo tags (gazebo_props:=false). -->
+    <xacro:include filename="$(find cra_description)/urdf/gripper.xacro"/>
+    <xacro:cr7_gripper gazebo_props="false"/>
     <!-- Import control_xacro -->
     <xacro:include filename="cr7_robot.ros2_control.xacro" />

File: src/DOBOT_6Axis_ROS2_V4/cra_description/urdf/cr7_on_mpo700.urdf.xacro (robot description, xacro)
@@ -351,106 +351,7 @@
     <selfCollide>true</selfCollide>
   </gazebo>
-  <!-- Blender fixed-jaw parallel gripper attached to Link6.
-       Flange mount face at z=+0.1401 in gripper frame (measured from mesh).
-       finger_joint axis -X: positive = opening, negative = closing. -->
-  <link name="gripper_base_link">
-    <inertial>
-      <origin xyz="0 0 0.05" rpy="0 0 0"/>
-      <mass value="0.8"/>
-      <inertia ixx="0.0060" ixy="0" ixz="0" iyy="0.0079" iyz="0" izz="0.0049"/>
-    </inertial>
-    <visual>
-      <origin xyz="0 0 0" rpy="0 0 0"/>
-      <geometry>
-        <mesh filename="file:///home/user/dobot_ws/src/blender/gripper/meshes/base.dae"/>
-      </geometry>
-    </visual>
-    <!-- Collision refit to hug base.dae visual parts (link frame, node tf applied).
-         Old primitives were phantom jaws reaching down to z=-0.116 where the visual
-         has nothing, pushing the shelf box without visual contact. The small side
-         tab (Cube_099) lies fully inside the body block, so it is omitted. -->
-    <!-- Fixed jaw (jaw_fixed + pad_fixed meshes) is C-shaped: a top beam plus
-         an outer column carrying the pad on its inner face. Two boxes that hug
-         those parts, leaving the grasp gap between the pads OPEN. The previous
-         single box was the whole jaw AABB: it filled the grasp gap with solid
-         collision, so the box was ejected on descend without visual contact. -->
-    <collision>  <!-- fixed-jaw top beam: X[0.009,0.107] Y[+-0.046] Z[0.105,0.115] -->
-      <origin xyz="0.0581 0 0.110" rpy="0 0 0"/>
-      <geometry><box size="0.098 0.0912 0.010"/></geometry>
-    </collision>
-    <collision>  <!-- fixed-jaw column + pad: X[0.0894,0.1071] Y[+-0.046] Z[0.055,0.105] -->
-      <origin xyz="0.0983 0 0.080" rpy="0 0 0"/>
-      <geometry><box size="0.0177 0.0912 0.050"/></geometry>
-    </collision>
-    <collision>  <!-- top plate (Cube_071): X[+-0.061] Y[+-0.046] Z[0.115,0.127] -->
-      <origin xyz="0 0 0.121" rpy="0 0 0"/>
-      <geometry><box size="0.121 0.091 0.012"/></geometry>
-    </collision>
-    <collision>  <!-- mount boss (Cylinder_004): r0.041 at Z[0.127,0.140] (flange face) -->
-      <origin xyz="0 0 0.134" rpy="0 0 0"/>
-      <geometry><cylinder radius="0.041" length="0.013"/></geometry>
-    </collision>
-  </link>
-  <joint name="gripper_attach_joint" type="fixed">
-    <origin xyz="0 0 0.1401" rpy="3.14159265359 0 0"/>
-    <parent link="Link6"/>
-    <child link="gripper_base_link"/>
-  </joint>
-  <link name="gripper_finger_link">
-    <inertial>
-      <origin xyz="-0.073 0 0.023" rpy="0 0 0"/>
-      <mass value="0.2"/>
-      <inertia ixx="0.0007" ixy="0" ixz="0" iyy="0.0005" iyz="0" izz="0.00035"/>
-    </inertial>
-    <visual>
-      <origin xyz="0 0 0" rpy="0 0 0"/>
-      <geometry>
-        <mesh filename="file:///home/user/dobot_ws/src/blender/gripper/meshes/finger.dae"/>
-      </geometry>
-    </visual>
-    <!-- Collision refit to finger.dae visual (Cube_096 jaw + Cube_100 tab) union AABB:
-         X[-0.011,0.016] Y[+-0.035] Z[0.056,0.127]. Old box (0.064x0.129x0.160 at
-         x=-0.073,z=0.023) was a phantom offset ~0.07 m in both X and Z from the
-         visual finger, which is what scraped the box during the insert. -->
-    <collision>
-      <origin xyz="0.0025 0 0.0915" rpy="0 0 0"/>
-      <geometry><box size="0.027 0.070 0.071"/></geometry>
-    </collision>
-  </link>
-  <joint name="gripper_finger_joint" type="prismatic">
-    <origin xyz="0 0 0" rpy="0 0 0"/>
-    <parent link="gripper_base_link"/>
-    <child link="gripper_finger_link"/>
-    <axis xyz="-1 0 0"/>
-    <limit lower="-0.07" upper="0.10" effort="60" velocity="0.1"/>
-    <dynamics damping="5.0" friction="1.0"/>
-  </joint>
-  <!-- Gazebo properties for the Blender gripper links -->
-  <gazebo reference="gripper_base_link">
-    <material>Gazebo/DarkGrey</material>
-    <gravity>false</gravity>
-    <!-- Soft contact like the finger below. Without these the fixed jaw uses
-         the Gazebo defaults (kp=1e12, maxVel=100): the moment the squeeze
-         presses the box into the fixed pad, the near-rigid contact fires a
-         huge impulse and shoots the box out of the grip. -->
-    <mu1>1.2</mu1>
-    <mu2>1.2</mu2>
-    <kp>1000000.0</kp>
-    <kd>1.0</kd>
-    <minDepth>0.001</minDepth>
-    <maxVel>0.1</maxVel>
-    <selfCollide>true</selfCollide>
-  </gazebo>
-  <gazebo reference="gripper_finger_link">
-    <material>Gazebo/Orange</material>
-    <gravity>false</gravity>
-    <mu1>1.2</mu1>
-    <mu2>1.2</mu2>
-    <kp>1000000.0</kp>
-    <kd>1.0</kd>
-    <minDepth>0.001</minDepth>
-    <maxVel>0.1</maxVel>
-    <selfCollide>true</selfCollide>
-  </gazebo>
+  <!-- Gripper: single source of truth in gripper.xacro (Gazebo sim -> gazebo_props on) -->
+  <xacro:include filename="$(find cra_description)/urdf/gripper.xacro"/>
+  <xacro:cr7_gripper/>
   <!-- ===================== CR7 ros2_control ===================== -->
   <ros2_control name="GazeboSystem" type="system">

File: src/DOBOT_6Axis_ROS2_V4/cra_description/urdf/cr7_robot.xacro (robot description, xacro)
@@ -426,91 +426,7 @@
         <selfCollide>true</selfCollide>
     </gazebo>
-    <!-- Blender fixed-jaw parallel gripper attached to Link6.
-         Flange mount face at z=+0.1443 in gripper frame; offset z=-0.1443 puts
-         that face at Link6's origin. finger_joint axis +X: positive = closing. -->
-    <link name="gripper_base_link">
-      <inertial>
-        <origin xyz="0 0 0.05" rpy="0 0 0"/>
-        <mass value="0.8"/>
-        <inertia ixx="0.0060" ixy="0" ixz="0" iyy="0.0079" iyz="0" izz="0.0049"/>
-      </inertial>
-      <visual>
-        <origin xyz="0 0 0" rpy="0 0 0"/>
-        <geometry>
-          <mesh filename="file:///home/user/dobot_ws/src/blender/gripper/meshes/base.dae"/>
-        </geometry>
-      </visual>
-      <collision>
-        <origin xyz="0 0 0.1336" rpy="0 0 0"/>
-        <geometry><cylinder radius="0.0675" length="0.0214"/></geometry>
-      </collision>
-      <collision>
-        <origin xyz="0 0 0.1129" rpy="0 0 0"/>
-        <geometry><box size="0.20 0.15 0.020"/></geometry>
-      </collision>
-      <collision>
-        <origin xyz="0.0125 0 0.0900" rpy="0 0 0"/>
-        <geometry><box size="0.225 0.15 0.0258"/></geometry>
-      </collision>
-      <collision>
-        <origin xyz="0.0510 0 -0.0193" rpy="0 0 0"/>
-        <geometry><box size="0.021 0.15 0.1928"/></geometry>
-      </collision>
-      <collision>
-        <origin xyz="0.0362 0 0.0071" rpy="0 0 0"/>
-        <geometry><box size="0.0086 0.14 0.12"/></geometry>
-      </collision>
-    </link>
-    <joint name="gripper_attach_joint" type="fixed">
-      <origin xyz="0 0 0.1443" rpy="3.14159265359 0 0"/>
-      <parent link="Link6"/>
-      <child link="gripper_base_link"/>
-    </joint>
-    <link name="gripper_finger_link">
-      <inertial>
-        <origin xyz="-0.073 0 0.023" rpy="0 0 0"/>
-        <mass value="0.2"/>
-        <inertia ixx="0.0007" ixy="0" ixz="0" iyy="0.0005" iyz="0" izz="0.00035"/>
-      </inertial>
-      <visual>
-        <origin xyz="0 0 0" rpy="0 0 0"/>
-        <geometry>
-          <mesh filename="file:///home/user/dobot_ws/src/blender/gripper/meshes/finger.dae"/>
-        </geometry>
-      </visual>
-      <collision>
-        <origin xyz="-0.0727 0 0.0229" rpy="0 0 0"/>
-        <geometry><box size="0.0643 0.1286 0.1601"/></geometry>
-      </collision>
-      <collision>
-        <origin xyz="-0.0362 0 0.0071" rpy="0 0 0"/>
-        <geometry><box size="0.0086 0.10 0.10"/></geometry>
-      </collision>
-    </link>
-    <joint name="gripper_finger_joint" type="prismatic">
-      <origin xyz="0 0 0" rpy="0 0 0"/>
-      <parent link="gripper_base_link"/>
-      <child link="gripper_finger_link"/>
-      <axis xyz="1 0 0"/>
-      <limit lower="-0.05" upper="0.07" effort="60" velocity="0.1"/>
-      <dynamics damping="5.0" friction="1.0"/>
-    </joint>
-    <!-- Gazebo properties for the Blender gripper links -->
-    <gazebo reference="gripper_base_link">
-        <material>Gazebo/DarkGrey</material>
-        <gravity>false</gravity>
-        <selfCollide>true</selfCollide>
-    </gazebo>
-    <gazebo reference="gripper_finger_link">
-        <material>Gazebo/Orange</material>
-        <gravity>false</gravity>
-        <mu1>1.2</mu1>
-        <mu2>1.2</mu2>
-        <kp>1000000.0</kp>
-        <kd>1.0</kd>
-        <minDepth>0.001</minDepth>
-        <maxVel>0.1</maxVel>
-        <selfCollide>true</selfCollide>
-    </gazebo>
+    <!-- Gripper: single source of truth in gripper.xacro (Gazebo sim -> gazebo_props on) -->
+    <xacro:include filename="$(find cra_description)/urdf/gripper.xacro"/>
+    <xacro:cr7_gripper/>
     <ros2_control name="GazeboSystem" type="system">
         <hardware>
@@ -579,9 +495,9 @@
         <joint name="gripper_finger_joint">
             <command_interface name="position">
-                <param name="min">-0.05</param>
-                <param name="max">0.07</param>
-            </command_interface>
-            <state_interface name="position">
-                <param name="initial_value">-0.04</param>
+                <param name="min">-0.07</param>
+                <param name="max">0.05</param>
+            </command_interface>
+            <state_interface name="position">
+                <param name="initial_value">0.04</param>
             </state_interface>
             <state_interface name="velocity"/>

File: src/DOBOT_6Axis_ROS2_V4/cra_description/urdf/gripper.xacro (robot description, xacro)
@@ -1,137 +1,97 @@
 <?xml version="1.0"?>
 <robot xmlns:xacro="http://www.ros.org/wiki/xacro">
-  <xacro:macro name="simple_gripper" params="parent prefix:='' *origin">
-    <xacro:property name="base_length"     value="0.060"/>
-    <xacro:property name="base_width"      value="0.080"/>
-    <xacro:property name="base_height"     value="0.050"/>
-    <xacro:property name="base_mass"       value="1.0"/>
-    <xacro:property name="finger_length"   value="0.080"/>
-    <xacro:property name="finger_width"    value="0.015"/>
-    <xacro:property name="finger_height"   value="0.030"/>
-    <xacro:property name="finger_mass"     value="0.25"/>
-    <xacro:property name="stroke_per_side" value="0.080"/>
-    <xacro:property name="initial_gap"     value="0.005"/>
-    <xacro:property name="max_effort"      value="100"/>
-    <xacro:property name="max_velocity"    value="0.15"/>
-    <xacro:macro name="box_inertia" params="m x y z">
+  <!-- Single source of truth for the Blender fixed-jaw parallel gripper on Link6.
+       Included by cr7_on_mpo700.urdf.xacro, cra_description/cr7_robot.xacro and
+       cr7_moveit/config/cr7_robot.urdf.xacro so the collision boxes stay in sync
+       (edit jaw geometry HERE only). Flange mount face at z=+0.1401; finger_joint
+       axis -X: positive = opening, negative = closing.
+       gazebo_props: emit the soft-contact + gravity-off Gazebo tags (true for the
+       Gazebo-sim robots; false for the MoveIt-only description, which has none). -->
+  <xacro:macro name="cr7_gripper" params="gazebo_props:=true">
+    <link name="gripper_base_link">
       <inertial>
+        <origin xyz="0 0 0.05" rpy="0 0 0"/>
+        <mass value="0.8"/>
+        <inertia ixx="0.0060" ixy="0" ixz="0" iyy="0.0079" iyz="0" izz="0.0049"/>
+      </inertial>
+      <visual>
         <origin xyz="0 0 0" rpy="0 0 0"/>
-        <mass value="${m}"/>
-        <inertia
-          ixx="${m*(y*y + z*z)/12}"
-          ixy="0" ixz="0"
-          iyy="${m*(x*x + z*z)/12}"
-          iyz="0"
-          izz="${m*(x*x + y*y)/12}"/>
+        <geometry>
+          <mesh filename="file:///home/user/dobot_ws/src/blender/gripper_long/meshes/base.dae"/>
+        </geometry>
+      </visual>
+      <!-- Fitted to gripper_long/meshes/base.dae per-part bounds (jaw_fixed, pad_fixed, body, flange) -->
+      <collision>  <!-- fixed-jaw top beam (jaw_fixed top): X[-0.021,0.181] Y[+-0.046] Z[0.105,0.115] -->
+        <origin xyz="0.0801 0 0.110" rpy="0 0 0"/>
+        <geometry><box size="0.2016 0.0912 0.010"/></geometry>
+      </collision>
+      <collision>  <!-- fixed-jaw column + contact pad: X[0.163,0.181] Y[+-0.046] Z[0.055,0.105], inner face = pad at X=0.1632 -->
+        <origin xyz="0.17205 0 0.080" rpy="0 0 0"/>
+        <geometry><box size="0.0177 0.0912 0.050"/></geometry>
+      </collision>
+      <collision>  <!-- top plate (body): X[-0.061,0.071] Y[+-0.046] Z[0.115,0.127] -->
+        <origin xyz="0.00505 0 0.12105" rpy="0 0 0"/>
+        <geometry><box size="0.1315 0.0912 0.0121"/></geometry>
+      </collision>
+      <collision>  <!-- mount boss (flange): r0.041 at Z[0.127,0.140] (flange face) -->
+        <origin xyz="0 0 0.13355" rpy="0 0 0"/>
+        <geometry><cylinder radius="0.041" length="0.013"/></geometry>
+      </collision>
+    </link>
+    <joint name="gripper_attach_joint" type="fixed">
+      <origin xyz="0 0 0.1401" rpy="3.14159265359 0 0"/>
+      <parent link="Link6"/>
+      <child link="gripper_base_link"/>
+    </joint>
+    <link name="gripper_finger_link">
+      <inertial>
+        <origin xyz="-0.073 0 0.023" rpy="0 0 0"/>
+        <mass value="0.2"/>
+        <inertia ixx="0.0007" ixy="0" ixz="0" iyy="0.0005" iyz="0" izz="0.00035"/>
       </inertial>
-    </xacro:macro>
-    <link name="${prefix}gripper_base">
       <visual>
-        <origin xyz="0 0 ${base_height/2}" rpy="0 0 0"/>
+        <origin xyz="0 0 0" rpy="0 0 0"/>
         <geometry>
-          <box size="${base_width} ${base_length} ${base_height}"/>
+          <mesh filename="file:///home/user/dobot_ws/src/blender/gripper_long/meshes/finger.dae"/>
         </geometry>
-        <material name="gripper_gray">
-          <color rgba="0.3 0.3 0.3 1.0"/>
-        </material>
       </visual>
-      <collision>
-        <origin xyz="0 0 ${base_height/2}" rpy="0 0 0"/>
-        <geometry>
-          <box size="${base_width} ${base_length} ${base_height}"/>
-        </geometry>
+      <collision>  <!-- moving jaw + contact pad (jaw_moving+pad_moving): X[0.055,0.082] Y[+-0.035] Z[0.056,0.127], outer face = pad at X=0.0822 -->
+        <origin xyz="0.0687 0 0.0916" rpy="0 0 0"/>
+        <geometry><box size="0.027 0.070 0.071"/></geometry>
       </collision>
-      <xacro:box_inertia m="${base_mass}" x="${base_width}" y="${base_length}" z="${base_height}"/>
     </link>
-    <joint name="${prefix}gripper_base_joint" type="fixed">
-      <xacro:insert_block name="origin"/>
-      <parent link="${parent}"/>
-      <child  link="${prefix}gripper_base"/>
+    <joint name="gripper_finger_joint" type="prismatic">
+      <origin xyz="0 0 0" rpy="0 0 0"/>
+      <parent link="gripper_base_link"/>
+      <child link="gripper_finger_link"/>
+      <axis xyz="-1 0 0"/>
+      <limit lower="-0.07" upper="0.10" effort="60" velocity="0.1"/>
+      <dynamics damping="5.0" friction="1.0"/>
     </joint>
-    <link name="${prefix}left_finger">
-      <visual>
-        <origin xyz="0 0 ${finger_length/2}" rpy="0 0 0"/>
-        <geometry>
-          <box size="${finger_width} ${finger_height} ${finger_length}"/>
-        </geometry>
-        <material name="finger_blue">
-          <color rgba="0.2 0.4 0.8 1.0"/>
-        </material>
-      </visual>
-      <collision>
-        <origin xyz="0 0 ${finger_length/2}" rpy="0 0 0"/>
-        <geometry>
-          <box size="${finger_width} ${finger_height} ${finger_length}"/>
-        </geometry>
-      </collision>
-      <xacro:box_inertia m="${finger_mass}" x="${finger_width}" y="${finger_height}" z="${finger_length}"/>
-    </link>
-    <joint name="${prefix}left_finger_joint" type="prismatic">
-      <origin xyz="${-(initial_gap/2 + finger_width/2)} 0 ${base_height}" rpy="0 0 0"/>
-      <parent link="${prefix}gripper_base"/>
-      <child  link="${prefix}left_finger"/>
-      <axis xyz="-1 0 0"/>
-      <limit lower="0.0" upper="${stroke_per_side}"
-             effort="${max_effort}" velocity="${max_velocity}"/>
-      <dynamics damping="10.0" friction="1.0"/>
-    </joint>
-    <link name="${prefix}right_finger">
-      <visual>
-        <origin xyz="0 0 ${finger_length/2}" rpy="0 0 0"/>
-        <geometry>
-          <box size="${finger_width} ${finger_height} ${finger_length}"/>
-        </geometry>
-        <material name="finger_blue">
-          <color rgba="0.2 0.4 0.8 1.0"/>
-        </material>
-      </visual>
-      <collision>
-        <origin xyz="0 0 ${finger_length/2}" rpy="0 0 0"/>
-        <geometry>
-          <box size="${finger_width} ${finger_height} ${finger_length}"/>
-        </geometry>
-      </collision>
-      <xacro:box_inertia m="${finger_mass}" x="${finger_width}" y="${finger_height}" z="${finger_length}"/>
-    </link>
-    <joint name="${prefix}right_finger_joint" type="prismatic">
-      <origin xyz="${initial_gap/2 + finger_width/2} 0 ${base_height}" rpy="0 0 0"/>
-      <parent link="${prefix}gripper_base"/>
-      <child  link="${prefix}right_finger"/>
-      <axis xyz="1 0 0"/>
-      <limit lower="0.0" upper="${stroke_per_side}"
-             effort="${max_effort}" velocity="${max_velocity}"/>
-      <dynamics damping="10.0" friction="1.0"/>
-      <mimic joint="${prefix}left_finger_joint" multiplier="1.0" offset="0.0"/>
-    </joint>
-    <link name="${prefix}tcp"/>
-    <joint name="${prefix}tcp_joint" type="fixed">
-      <origin xyz="0 0 ${base_height + finger_length}" rpy="0 0 0"/>
-      <parent link="${prefix}gripper_base"/>
-      <child  link="${prefix}tcp"/>
-    </joint>
-    <gazebo reference="${prefix}gripper_base">
-      <material>Gazebo/DarkGrey</material>
-      <gravity>false</gravity>
-    </gazebo>
-    <gazebo reference="${prefix}left_finger">
-      <material>Gazebo/Blue</material>
-      <gravity>false</gravity>
-      <mu1>2.0</mu1>
-      <mu2>2.0</mu2>
-      <kp>1000000.0</kp>
-      <kd>1.0</kd>
-      <minDepth>0.001</minDepth>
-      <maxVel>0.1</maxVel>
-    </gazebo>
-    <gazebo reference="${prefix}right_finger">
-      <material>Gazebo/Blue</material>
-      <gravity>false</gravity>
-      <mu1>2.0</mu1>
-      <mu2>2.0</mu2>
-      <kp>1000000.0</kp>
-      <kd>1.0</kd>
-      <minDepth>0.001</minDepth>
-      <maxVel>0.1</maxVel>
-    </gazebo>
+    <xacro:if value="${gazebo_props}">
+      <!-- Soft contact so the squeeze doesn't fire a huge impulse and eject the box -->
+      <gazebo reference="gripper_base_link">
+        <material>Gazebo/DarkGrey</material>
+        <gravity>false</gravity>
+        <mu1>1.2</mu1>
+        <mu2>1.2</mu2>
+        <kp>1000000.0</kp>
+        <kd>1.0</kd>
+        <minDepth>0.001</minDepth>
+        <maxVel>0.1</maxVel>
+        <selfCollide>true</selfCollide>
+      </gazebo>
+      <gazebo reference="gripper_finger_link">
+        <material>Gazebo/Orange</material>
+        <gravity>false</gravity>
+        <mu1>1.2</mu1>
+        <mu2>1.2</mu2>
+        <kp>1000000.0</kp>
+        <kd>1.0</kd>
+        <minDepth>0.001</minDepth>
+        <maxVel>0.1</maxVel>
+        <selfCollide>true</selfCollide>
+      </gazebo>
+    </xacro:if>
   </xacro:macro>
 </robot>
